Commit message: fix: add robot models in packag

File: urdf/robot1_base_04.xacro (robot description, xacro)
@@ -25,5 +25,7 @@
 		<xacro:default_inertial mass="0.0001"/>
  	</link>
- 	<xacro:include filename="$(find robot1_description)/urdf/robot.gazebo" />
+	<!--what is this???? robot.gazebo??? material properties for robot model-->
+ 	<!--xacro:include filename="$(find robot1_description)/urdf/robot.gazebo" /-->
+	<xacro:include filename="$(find learning_nav)/robot_models/robot.gazebo" />
 	<gazebo reference="base_footprint">
 		<material>Gazebo/Green</material>
@@ -192,5 +194,6 @@
       <origin xyz="0 0 0" rpy="0 0 0"/>
       <geometry>
-        <mesh filename="package://robot1_description/meshes/hokuyo.dae"/>
+        <!--mesh filename="package://robot1_description/meshes/hokuyo.dae"/-->
+				<mesh filename="package://learning_nav/robot_models/hokuyo.dae"/>
       </geometry>
     </visual>
